File: LED-Board/BloopBox LED-Board.kicad_pcb (KiCad board)
At the start: 2 copper layers, 25 x 15 mm, 4 parts, among them J1 Mainboard

Commit message: fix(LED-Board): make sure ERC works
Connections:
- net +5V renamed /+5V
Changed lines of the file:
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@@
   )
   (setup
+    (stackup
+      (layer "F.SilkS" (type "Top Silk Screen"))
+      (layer "F.Paste" (type "Top Solder Paste"))
+      (layer "F.Mask" (type "Top Solder Mask") (thickness 0.01))
+      (layer "F.Cu" (type "copper") (thickness 0.035))
+      (layer "dielectric 1" (type "core") (thickness 1.51) (material "FR4") (epsilon_r 4.5) (loss_tangent 0.02))
+      (layer "B.Cu" (type "copper") (thickness 0.035))
+      (layer "B.Mask" (type "Bottom Solder Mask") (thickness 0.01))
+      (layer "B.Paste" (type "Bottom Solder Paste"))
+      (layer "B.SilkS" (type "Bottom Silk Screen"))
+      (copper_finish "None")
+      (dielectric_constraints no)
+    )
     (pad_to_mask_clearance 0)
     (pcbplotparams
@@
   (net 0 "")
   (net 1 "/R")
-  (net 2 "+5V")
+  (net 2 "/+5V")
   (net 3 "/G")
   (net 4 "/B")
@@
     (descr "Mounting Hole 3.2mm, M3")
     (tags "mounting hole 3.2mm m3")
-    (property "Sheetfile" "LED-Board.kicad_sch")
+    (property "Sheetfile" "BloopBox LED-Board.kicad_sch")
     (property "Sheetname" "")
     (attr exclude_from_pos_files)
@@
     (descr "Mounting Hole 3.2mm, M3")
     (tags "mounting hole 3.2mm m3")
-    (property "Sheetfile" "LED-Board.kicad_sch")
+    (property "Sheetfile" "BloopBox LED-Board.kicad_sch")
     (property "Sheetname" "")
     (attr exclude_from_pos_files)
@@
     (descr "LED, diameter 5.0mm, 4 pins, WP154A4, https://www.kingbright.com/attachments/file/psearch/000/00/00/L-154A4SUREQBFZGEW(Ver.11A).pdf")
     (tags "rgb led")
-    (property "Sheetfile" "LED-Board.kicad_sch")
+    (property "Sheetfile" "BloopBox LED-Board.kicad_sch")
     (property "Sheetname" "")
     (attr through_hole)
@@
       (net 1 "/R") (pinfunction "RK") (pintype "passive"))
     (pad "2" thru_hole circle (at -0.635 0.762) (size 1.8 1.8) (drill 0.9) (layers *.Cu *.Mask)
-      (net 2 "+5V") (pinfunction "A") (pintype "passive"))
+      (net 2 "/+5V") (pinfunction "A") (pintype "passive"))
     (pad "3" thru_hole circle (at 0.889 -0.762) (size 1.8 1.8) (drill 0.9) (layers *.Cu *.Mask)
       (net 3 "/G") (pinfunction "GK") (pintype "passive"))
@@
     (descr "JST PH series connector, S4B-PH-K (http://www.jst-mfg.com/product/pdf/eng/ePH.pdf), generated with kicad-footprint-generator")
     (tags "connector JST PH top entry")
-    (property "Sheetfile" "LED-Board.kicad_sch")
+    (property "Sheetfile" "BloopBox LED-Board.kicad_sch")
     (property "Sheetname" "")
     (attr through_hole)
@@
       (net 3 "/G") (pinfunction "Pin_2") (pintype "passive"))
     (pad "3" thru_hole oval (at 4 0 180) (size 1.2 1.75) (drill 0.75) (layers *.Cu *.Mask)
-      (net 2 "+5V") (pinfunction "Pin_3") (pintype "passive"))
+      (net 2 "/+5V") (pinfunction "Pin_3") (pintype "passive"))
     (pad "4" thru_hole oval (at 6 0 180) (size 1.2 1.75) (drill 0.75) (layers *.Cu *.Mask)
       (net 1 "/R") (pinfunction "Pin_4") (pintype "passive"))
